File: pcb/esp32-s2/esp32-s2.kicad_pcb (KiCad board)
At the start: 2 copper layers, 40.4 x 33.8 mm, 31 parts, among them J1 BATT, J2 HALL-CONN, Q1 BC817, Q2 BC807, SW2 RST, U1 XC6220, U2 ESP32-S2-WROOM

Commit message: add todo
Parts:
- C1: value C -> 22µF
- C2: value C -> 4,7µF
Connections:
- net Net-(R1-Pad2) renamed /IO18
